Commit message: update

File: source/isaaclab_tasks/isaaclab_tasks/direct/np/asset/mesh/frame_back_rod_rod.urdf (robot description, URDF)
Before this commit: robot frame_back, 10 links, 9 joints
Links:
- link plug1: geometry collision mesh filename=plug.obj scale=0.6 0.6 0.75; visual mesh filename=plug.obj scale=0.6 0.6 0.75
- link plug2: geometry collision mesh filename=plug.obj scale=0.6 0.6 0.75; visual mesh filename=plug.obj scale=0.6 0.6 0.75
- link plug3: geometry collision mesh filename=plug.obj scale=0.6 0.6 0.75; visual mesh filename=plug.obj scale=0.6 0.6 0.75
- link plug4: geometry collision mesh filename=plug.obj scale=0.6 0.6 0.75; visual mesh filename=plug.obj scale=0.6 0.6 0.75
- link plug5: geometry collision mesh filename=plug.obj scale=0.6 0.6 0.75; visual mesh filename=plug.obj scale=0.6 0.6 0.75
- link plug6: geometry collision mesh filename=plug.obj scale=0.6 0.6 0.75; visual mesh filename=plug.obj scale=0.6 0.6 0.75
Joints:
- joint frame_to_plug1: origin xyz=0.0174 0.228 -0.45 rpy=1.5708 0 3.1416 -> xyz=0.016 0.228 -0.448 rpy=1.5708 0 3.1416
- joint frame_to_plug2: origin xyz=0.0174 0.228 -0.417 rpy=1.5708 0 3.1416 -> xyz=0.016 0.228 -0.416 rpy=1.5708 0 3.1416

Commit message: finish chair4

File: source/isaaclab_tasks/isaaclab_tasks/direct/np/asset/mesh/frame_back_rod_rod.urdf (robot description, URDF)
Before this commit: robot frame_back, 10 links, 9 joints
Links:
- link plug1: geometry collision mesh filename=plug.obj scale=0.4 0.4 0.75; visual mesh filename=plug.obj scale=0.6 0.6 0.75
- link plug2: geometry collision mesh filename=plug.obj scale=0.4 0.4 0.75; visual mesh filename=plug.obj scale=0.6 0.6 0.75
- link plug3: geometry collision mesh filename=plug.obj scale=0.4 0.4 0.75; visual mesh filename=plug.obj scale=0.6 0.6 0.75
- link plug4: geometry collision mesh filename=plug.obj scale=0.4 0.4 0.75; visual mesh filename=plug.obj scale=0.6 0.6 0.75
- link plug5: geometry collision mesh filename=plug.obj scale=0.4 0.4 0.75; visual mesh filename=plug.obj scale=0.6 0.6 0.75
- link plug6: geometry collision mesh filename=plug.obj scale=0.4 0.4 0.75; visual mesh filename=plug.obj scale=0.6 0.6 0.75
