Commit message: update chair5_1

File: source/isaaclab_tasks/isaaclab_tasks/direct/np/asset/mesh/chair_all.urdf (robot description, URDF)
Before this commit: robot frame_back, 5 links, 4 joints
Links:
- added link seat, mass 1.0; collision mesh filename=seat.obj; visual mesh filename=seat.obj
Joints:
- added joint frame_to_seat: type fixed, parent frame_re, child seat, origin xyz=0.0031 0.26 -0.27 rpy=-3.1415 3.1415 1.5708
